File: STM32_Sensor_V4.sch (KiCad schematic (older format))
At the start: 26 parts, among them J1 Conn Side, J2 Conn Down, J3 Conn Up, J4 Conn Prog, J5 u.FL, SW1 SW_Reset, SW2 SW_BOOT, U1 STM32F103C8Tx, U2 RFM69CW, U3 RFM69HW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

Commit message: Added support for RFM69HCW
Previously only RFM69CW and RFM69(H)W were supported.
Parts:
- added U4: RFM69HCW, custom:RFM69HCW-XXXS2-MINPADS, symbol RF_AM_FM:RFM69HCW
- U2: footprint RF:RFM69CW-XXXS2 -> custom:RFM69CW-XXXS2-MINPADS
- U3: footprint RF_Module:HOPERF_RFM69HW -> custom:HOPERF_RFM69HW-MINPADS
Connections:
- wire segments 130 -> 101
- no-connect marks 9 -> 14
