File: STM32_Sensor.sch (KiCad schematic (older format))
At the start: 27 parts, among them J1 Conn Side, J2 Conn Down, J3 Conn Up, J4 Conn Prog, J5 u.FL, SW1 SW_Reset, SW2 SW_BOOT, U1 STM32F103C8Tx, U2 RFM69CW, U3 RFM69HW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

Commit message: Made VBAT jumper NO
to comply with PCB manufacturer design rules.
Parts:
- JP1: footprint Jumper:SolderJumper-2_P1.3mm_Bridged_Pad1.0x1.5mm -> Sparkfun Jumpers:SMT-JUMPER_2_NO_NO-SILK
Changed lines of the file:
@@
 EESchema Schematic File Version 4
-LIBS:STM32_Sensor_V4-cache
 EELAYER 26 0
 EELAYER END
@@
 F 0 "JP1" H 4510 3545 50  0000 C CNN
 F 1 "VBAT Jumper" H 4510 3454 50  0000 C CNN
-F 2 "Jumper:SolderJumper-2_P1.3mm_Bridged_Pad1.0x1.5mm" H 4510 3340 50  0001 C CNN
+F 2 "Sparkfun Jumpers:SMT-JUMPER_2_NO_NO-SILK" H 4510 3340 50  0001 C CNN
 F 3 "~" H 4510 3340 50  0001 C CNN
 	1    4510 3340
